File: teensy-tinyfpga.sch (KiCad schematic (older format))
At the start: 62 parts

Commit message: add footprints
Parts:
- C1, C10, C11, C12, C13, C14, C15, C17, C18, C19, C2, C20, C21, C22, C23, C24, C25, C26, C27, C28, C29, C3, C30, C31, C32, C33, C34, C35, C36, C37, C38, C39, C4, C40, C41, C42, C43, C44, C5, C6, C7, C8, C9: renamed from C?; footprint (none) -> Capacitor_SMD:C_0805_2012Metric
- FB1: renamed from FB?; footprint (none) -> Inductor_SMD:L_0603_1608Metric
- J1: renamed from J?; footprint (none) -> Connector_PinHeader_2.54mm:PinHeader_1x08_P2.54mm_Vertical
- J2, J3: renamed from J?; footprint (none) -> Connector_PinHeader_2.00mm:PinHeader_2x08_P2.00mm_Vertical
- R1, R3, R4: renamed from R?; value R -> 2k; footprint (none) -> Resistor_SMD:R_0805_2012Metric
- R2: renamed from R?; footprint (none) -> Resistor_SMD:R_0805_2012Metric
- R5, R6, R7: renamed from R?; value R -> 4.7k; footprint (none) -> Resistor_SMD:R_0805_2012Metric
- U1, U6: renamed from U?; footprint (none) -> Package_QFP:LQFP-64_10x10mm_P0.5mm
- U2, U3: renamed from U?; footprint (none) -> Package_SO:HTSSOP-24-1EP_4.4x7.8mm_P0.65mm_EP3.2x5mm
- U4: renamed from U?; footprint (none) -> footprints:Teensy41
- U7: renamed from U?; footprint (none) -> footprints:TinyFPGA_BX
- gave numbers to parts that had none: 2
Other:
- note added: "ST3375 TFT"
